Commit message: feat(localization): add dual-tag UWB yaw estimation pipeline

File: ros2_uwb_research_sim/urdf/robot.urdf (robot description, URDF)
Before this commit: robot tag_robot, 4 links, 3 joints
Links:
- added link front_tag; visual sphere radius=0.05
- added link rear_tag; visual sphere radius=0.05
Joints:
- added joint front_tag_joint: type fixed, parent base_link, child front_tag, origin xyz=0.35 0 0.1 rpy=0 0 0
- added joint rear_tag_joint: type fixed, parent base_link, child rear_tag, origin xyz=-0.35 0 0.1 rpy=0 0 0
